Commit message: mission complete

File: gazebo_environment/turtlebot3_description/urdf/turtlebot3_waffle.urdf.xacro (robot description, xacro)
@@ -7,5 +7,5 @@
     <parent link="base_footprint"/>
     <child link="base_link" />
-    <origin xyz="0 0 0.010" rpy="0 0 0"/>
+    <origin xyz="0.5 2 0.010" rpy="0 0 0"/>
   </joint>
   <link name="base_link">

Commit message: small change

File: gazebo_environment/turtlebot3_description/urdf/turtlebot3_waffle.urdf.xacro (robot description, xacro)
@@ -7,5 +7,5 @@
     <parent link="base_footprint"/>
     <child link="base_link" />
-    <origin xyz="0.5 2 0.010" rpy="0 0 0"/>
+    <origin xyz="0.0 0.0 0.0" rpy="0 0 0"/>
   </joint>
   <link name="base_link">
